File: ELEKTRA-PMIC/V0.1/ELEKTRA-PMIC v0.1-20240112.brd (EAGLE design)
At the start: 40 x 27 mm, 93 parts, among them U1 BQ24195L, U4 MAX1704X

Commit message: upload PCB and sch
upload PCB and sch
Parts:
- L1: value 1.5uH -> 2.2uH
- L3: value 1uH -> 2.2uH
- R11: value NC -> 0R
- R15: value NC -> 1nF
- R16, R23: value NC -> 1M
- R17: value 511K -> 24K
- R18, R24: value 1M -> NC
- R22: value NC -> 4.7uF
- R34: value 31.23K -> 31.2K
- R35: value 5.52K -> 5.49K
- R4: value 511K -> 1.1M
- R5, R9: value 91K -> 180K
- R6: value 511K -> 62K
- R8: value 511K -> 1M
Other:
- board text added: "R16（NC）/R18(1M)-贴片对调-R16（1M）/R18(NC)-此图是正确位置"
- board text added: "R23（NC）/R24(1M)-贴片对调-R23（1M）/R24(NC)"
- board text added: "添加"
