File: ELEKTRA-PMIC/V0.1/ELEKTRA-PMIC v0.1-20240112.sch (EAGLE design)
At the start: 93 parts, among them U1 BQ24195L, U4 MAX1704X

Commit message: upload PCB and sch
upload PCB and sch
Parts:
- L1: value 1.5uH -> 2.2uH
- L3: value 1uH -> 2.2uH
- R11: value NC -> 0R
- R15: value NC -> 1nF
- R16, R23: value NC -> 1M
- R17: value 511K -> 24K
- R18, R24: value 1M -> NC
- R22: value NC -> 4.7uF
- R34: value 31.23K -> 31.2K
- R35: value 5.52K -> 5.49K
- R4: value 511K -> 1.1M
- R5, R9: value 91K -> 180K
- R6: value 511K -> 62K
- R8: value 511K -> 1M
Other:
- note added: "R1up = R2down(VOUT/VFB - 1 ). VFB=0.5V"
