File: ELEKTRA-PMIC/v0.2-layout/ELEKTRA-PMIC v0.2-35X22.86-0.8.sch (EAGLE design)
At the start: 96 parts, among them U1 BQ24195L, U4 MAX1704X

Commit message: update layout
complete the layout for power module
Parts:
- removed JP1: M12PTH-CST-R, Particle:M12PTH-CST-R
- removed TP20, TP21, TP22: TP0.4MM, particle SZ:TP0.4MM
- removed U$1: M13PTH-CST-R, Particle:M13PTH-CST-R
- added J1: M13PTH-CST-R, Particle:M13PTH-CST-R
- added J2: M12PTH-CST-R, Particle:M12PTH-CST-R
- C101: value CAP-ECASE_B -> 220uF.6V
- C102: value CAP-ECASE_B -> 220uF,6V
- TP10, TP11, TP3, TP4, TP5, TP6, TP7, TP8, TP9: value TP -> TP0.4MM; device particle SZ:TP -> particle SZ:TP0.4MM
- renumbered U$4 to C101, U$5 to C102, U$6 to U6
Connections:
- removed net PMID: JP1.8
- net !FUEL-INT: now also J1.4; no longer U$1.4
- net !RST: now also J1.11; no longer U$1.11
- net 3V3: now also J2.1, J2.2; no longer JP1.1, JP1.2
- net 5VDC: now also J2.3, J2.4; no longer JP1.3, JP1.4
- net CHG: now also J1.1; no longer U$1.1
- net ENABLE: now also J1.13; no longer U$1.13
- net GND: now also J1.10, J1.9, J2.10, J2.9; no longer JP1.10, JP1.9, TP20.1, TP21.1, TP22.1, U$1.10, U$1.9
- net PG: now also J1.12; no longer U$1.12
- net REGN: now also J2.7; no longer JP1.7
- net SCL: now also J1.2; no longer U$1.2
- net SDA: now also J1.3; no longer U$1.3
- net TS: now also J1.5; no longer U$1.5
- net VBAT: now also J1.6, J1.7, J1.8; no longer U$1.6, U$1.7, U$1.8
- net VCC: now also J2.5, J2.6; no longer JP1.5, JP1.6
- net VIN: now also J2.11, J2.12; no longer JP1.11, JP1.12
Other:
- moved on the sheet: TP10, TP11, TP12, TP13, TP14, TP15, TP16, TP17, TP18, TP19, TP3, TP4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

Commit message: update layout
Optimize routing
Parts:
- removed C10: 100pF, Particle:CAP_1
- removed R1: 0R, Spark:R-US_
- added R34: 31.2K, Spark:R-US_
- added R35: 5.49K, Spark:R-US_
- R14: value 1M -> 100K
- TP1, TP2: value TPTP -> TP1311MM; device particle SZ:TPTP -> particle SZ:TP1311MM
Connections:
- removed net N$1: R1.1, U1.!QON
- net GND: now also R34.2; no longer C10.P$1
- net REGN: now also R35.1
- net TS: now also R34.1, R35.2, U1.!QON; no longer R1.2
- net VIN: no longer C10.P$2
