File: PowerModule_TestBoard/eagle/PowerModule_Testboard.brd (EAGLE design)
At the start: 160 x 100 mm, 30 parts, among them J1 1X2-3.5MM, J2 1X2-3.5MM, J9 1X2-3.5MM

Commit message: update the power module
Parts:
- removed J9: 1X2-3.5MM, adafruit:1X2-3.5MM
- added D1: (no value), particle-studios:SOD-123FL
- added J12: TP_OPEN, particle SZ:TP_OPEN
- added J3: (no value), particle-studios:JST-3-SMD-VERT
- added J5: 1X2-3.5MM, adafruit:1X2-3.5MM
- added JP3: (no value), microbuilder:JUMPER2
- added LED1: (no value), adafruit:CHIP-LED0603
- added R1, R2, R3, R4: 10K, particle-studios:R0603_P
- added R10, R9: 5K1, particle-studios:R0603_P
- added R5: 2K, particle-studios:R0603_P
- added USB1: (no value), SparkFun-Connectors:USB-C-16P
- J2: value 1X2-3.5MM -> (none); device adafruit:1X2-3.5MM -> SparkFun-Connectors:JST-2-SMD@2
- J4: value (none) -> 1X2-3.5MM; device SparkFun-Connectors:JST-2-SMD -> adafruit:1X2-3.5MM
- moved C10 285.6 mm to (67.6, 34.7), turned to 180 degrees
- moved SV1 262.5 mm to (76.2, 18.4), turned to 270 degrees
- moved J4 230.3 mm to (3.81, 45.7), turned to 90 degrees
- moved S4 227.4 mm to (46.5, 55.2), turned to 270 degrees
- moved R19 226.5 mm to (42.9, 51.7)
- moved R13 207.3 mm to (56.5, 12.1)
- moved LED3 200.9 mm to (59.1, 12.1), turned to 270 degrees
- moved JP7 200.3 mm to (54.0, 12.1)
- moved JP9 178.8 mm to (14.6, 47.0), turned to 270 degrees
- moved TP6 173.4 mm to (9.53, 47.6), turned to 270 degrees
- moved JP1 168.7 mm to (14.6, 31.5), turned to 90 degrees
- moved JP2 163.4 mm to (14.6, 21.0), turned to 270 degrees
- moved TP4 146.8 mm to (9.53, 30.5), turned to 270 degrees
- moved TP3 145.5 mm to (9.53, 34.3), turned to 90 degrees
- moved TP5 139.4 mm to (9.53, 17.8), turned to 90 degrees
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Connections:
- net N$2 renamed V_MODEM
- removed net N$10: C10.1, J4.1, U$2.21, U$2.22
- removed net N$14: C10.2, J4.2, U$2.18, U$2.19, U$2.20
- removed net N$16: SV1.10, U$2.28
- new net +5V: D1.A, USB1.VBUS1, USB1.VBUS2
- new net CC1: R10.2, USB1.A5
- new net CC2: R9.2, USB1.B5
- new net N$2: R19.2, S4.2, S4.5
- new net USB_N: SV1.10, U$2.28, USB1.A7, USB1.B7
- new net USB_P: SV1.9, U$2.29, USB1.A6, USB1.B6
- new net VBATT: C10.2, J2.2, J3.3, U$2.18, U$2.19, U$2.20
- new net VIN: C7.+, C8.1, C9.1, D1.C, J5.2, JP2.1, TP5.1, U$2.11, U$2.12
- net +3V3: now also J4.2, R3.2, R5.1; no longer J9.1, R19.2
- net GND: now also C10.1, J2.1, J3.2, J4.1, J5.1, LED1.C, R10.1, R19.1, R2.1, R4.1, R9.1, U$2.21, U$2.22, USB1.GND, USB1.GND2, USB1.SHLD1, USB1.SHLD2, USB1.SHLD3, USB1.SHLD4, USB1.SHLD5, USB1.SHLD6, USB1.SHLD7, USB1.SHLD8; no longer J2.2, J9.2
- net N$15: now also LED1.A, R5.2; no longer SV1.9, U$2.29
- net N$3: now also J12.1, R1.1, R2.2; no longer C7.+, C8.1, C9.1, J2.1, JP2.1, TP5.1, U$2.11, U$2.12
- net N$4: now also R3.1
- net N$5: now also J12.2, J3.1, JP3.1
- net N$9: now also JP3.2, R4.2; no longer R19.1, S4.2, S4.5
- net PMIC_REG: now also R1.2
Routing:
- net +3V3: track 0.00 -> 163.7 mm, vias 0 -> 1
- net GND: track 0.00 -> 94.6 mm, vias 0 -> 147
- net USB_N: track 0.00 -> 84.3 mm, vias 0 -> 2
- net USB_P: track 0.00 -> 80.3 mm, vias 0 -> 2
- net N$5: track 0.00 -> 38.2 mm
- net N$13: track 0.00 -> 37.9 mm, vias 0 -> 1
- net N$4: track 0.00 -> 24.6 mm, vias 0 -> 1
- net N$11: track 0.00 -> 22.2 mm
- net N$6: track 0.00 -> 17.8 mm
- net N$8: track 0.00 -> 17.8 mm
- net N$7: track 0.00 -> 17.7 mm
- net +5V: track 0.00 -> 16.9 mm
- net N$3: track 0.00 -> 11.4 mm
- net N$2: track 0.00 -> 10.0 mm
- net VIN: track 0.00 -> 8.38 mm
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- added copper zone on layer 1, net +3V3
- added copper zone on layer 1, net GND
- added copper zone on layer 16, net GND
- added copper zone on layer 1, net VBATT
- added copper zone on layer 1, net VIN
- added copper zone on layer 1, net V_MODEM
Other:
- board size 160 x 100 mm -> 80 x 57.1 mm
- board text added: "!PMIC_INT"
- board text added: "!PMIC_PG"
- board text added: "+"
- board text added: "+3.3V"
- board text added: "-"
- board text added: "3.3V"
- board text added: "CHARGE"
- board text added: "CHARGE STATE"
- board text added: "EN"
- board text added: "GND"
- board text added: "NTC"
- board text added: "OFF"
- board text added: "ON"
- board text added: "PMIC_REG"
- board text added: "PMIC_TS"
- board text added: "Power module EVB v0.0.1"
- board text added: "SCL"
- board text added: "SDA"
- board text added: "USB_N"
- board text added: "USB_P"
- board text added: "VIN"
- board text added: "V_MODEM"
