File: PowerModule_TestBoard/eagle/PowerModule_Testboard.sch (EAGLE design)
At the start: 30 parts, among them J1 1X2-3.5MM, J2 1X2-3.5MM, J9 1X2-3.5MM

Commit message: update the power module
Parts:
- removed J9: 1X2-3.5MM, adafruit:1X2-3.5MM
- added D1: (no value), particle-studios:DIODE_SOD-123FL
- added J12: TP_OPEN, particle SZ:TP_OPEN
- added J3: (no value), particle-studios:CONN_03JST-SMD-VERT
- added J5: 1X2-3.5MM, adafruit:1X2-3.5MM
- added JP3: (no value), microbuilder:JUMPER2
- added LED1: (no value), adafruit:LEDCHIP-LED0603
- added R1, R2, R3, R4: 10K, particle-studios:RES_100K_0603
- added R10, R9: 5K1, particle-studios:RES_0603
- added R5: 2K, particle-studios:RES_2K2_0603
- added USB1: (no value), SparkFun-Connectors:USB_C16PIN
- J2: value 1X2-3.5MM -> (none); device adafruit:1X2-3.5MM -> SparkFun-Connectors:CONN_02-JST-2MM-SMT
- J4: value (none) -> 1X2-3.5MM; device SparkFun-Connectors:CONN_02-JST-2MM-SMT -> adafruit:1X2-3.5MM
Connections:
- net N$2 renamed V_MODEM
- removed net N$10: C10.1, J4.2, U$2.GND@3, U$2.GND@4
- removed net N$14: C10.2, J4.1, U$2.V_BAT@1, U$2.V_BAT@2, U$2.V_BAT@3
- removed net N$16: SV1.10, U$2.PMIC_USB_DM
- new net +5V: D1.A, USB1.VBUS
- new net CC1: R10.2, USB1.CC1
- new net CC2: R9.2, USB1.CC2
- new net N$2: R19.2, S4.2, S4.5
- new net USB_N: SV1.10, U$2.PMIC_USB_DM, USB1.D-
- new net USB_P: SV1.9, U$2.PMIC_USB_DP, USB1.D+
- new net VBATT: C10.2, J2.1, J3.3, U$2.V_BAT@1, U$2.V_BAT@2, U$2.V_BAT@3
- new net VIN: C7.+, C8.1, C9.1, D1.C, J5.2, JP2.1, TP5.TP, U$2.VIN@1, U$2.VIN@2
- net +3V3: now also J4.2, R3.2, R5.1; no longer J9.1, R19.2
- net GND: now also C10.1, J3.2, J4.1, J5.1, LED1.C, R10.1, R19.1, R2.1, R4.1, R9.1, U$2.GND@3, U$2.GND@4, USB1.GND, USB1.SHLD; no longer J9.2
- net N$15: now also LED1.A, R5.2; no longer SV1.9, U$2.PMIC_USB_DP
- net N$3: now also J12.1, R1.1, R2.2; no longer C7.+, C8.1, C9.1, J2.1, JP2.1, TP5.TP, U$2.VIN@1, U$2.VIN@2
- net N$4: now also R3.1
- net N$5: now also J12.2, J3.1, JP3.1
- net N$9: now also JP3.2, R4.2; no longer R19.1, S4.2, S4.5
- net PMIC_REG: now also R1.2
Other:
- note added: "USB C CONNECTOR"
- moved on the sheet: R19
