File: PowerModule_TestBoard/eagle/powerModule_v0.0.2/PowerModule_Testboard_v0.0.2.sch (EAGLE design)
At the start: 43 parts, among them J1 1X2-3.5MM, J12 TP_OPEN, J4 1X2-3.5MM, J5 1X2-3.5MM

Commit message: update the design file
Parts:
- U$2: value PARTICLE_POWER_MODULE_SMT -> PARTICLE_POWER_MODULE; device particle-studios:PARTICLE_POWER_MODULE_SMT -> particle-studios:PARTICLE_POWER_MODULE
Other:
- moved on the sheet: C1, C10, C2, C3, C4, C5, C6, C7, C8, C9, D1, J12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

Commit message: update the power module v0.0.2
Connections:
- removed net PMIC_REG: R1.2, SV1.3
- net PMIC_RGEN: now also R1.2, SV1.3
Changed lines of the file:
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@@
 <pinref part="U$2" gate="G$1" pin="PMIC_RGEN"/>
+</segment>
+<segment>
+<pinref part="SV1" gate="1" pin="3"/>
+<wire x1="174.625" y1="113.03" x2="159.385" y2="113.03" width="0.1524" layer="91"/>
+<label x="159.385" y="113.03" size="1.016" layer="95"/>
+<pinref part="R1" gate="R1" pin="2"/>
+<wire x1="216.535" y1="104.14" x2="216.535" y2="113.03" width="0.1524" layer="91"/>
+<wire x1="216.535" y1="113.03" x2="174.625" y2="113.03" width="0.1524" layer="91"/>
+<junction x="174.625" y="113.03"/>
 </segment>
 </net>
@@
 </segment>
 </net>
-<net name="PMIC_REG" class="0">
-<segment>
-<pinref part="SV1" gate="1" pin="3"/>
-<wire x1="174.625" y1="113.03" x2="159.385" y2="113.03" width="0.1524" layer="91"/>
-<label x="159.385" y="113.03" size="1.016" layer="95"/>
-<pinref part="R1" gate="R1" pin="2"/>
-<wire x1="216.535" y1="104.14" x2="216.535" y2="113.03" width="0.1524" layer="91"/>
-<wire x1="216.535" y1="113.03" x2="174.625" y2="113.03" width="0.1524" layer="91"/>
-<junction x="174.625" y="113.03"/>
-</segment>
-</net>
