File: PM-BAT/V0.1/PM-BAT/v0.2-layout/ELEKTRA-PMIC v0.2-35X22.86-0.8.sch (EAGLE design)
At the start: 87 parts, among them J1 M13PTH-CST-R, J2 M12PTH-CST-R, U1 BQ24195, U2 TPS63020, U3 TPS631011, U4 MAX1704X, U5 TPS22918

Commit message: update
change the name as PM-BAT
Parts:
- removed C10: 0.1uF, particle SZ:CAPC0201-N
- removed C7: 1000pF,25V, particle SZ:CAP0402A
- removed R1: 100K, particle SZ:RESR0201-N
- removed R11: 10K, particle SZ:RESR0201-N
- removed R12: 10K/NC, particle SZ:RESR0201-N
- removed R13: 100K/NC, particle SZ:RESR0201-N
- removed U$1, U$2, U$4, U$5: TP, Particle:TP
- removed U5: TPS22918, particle SZ:TPS22918
- added TP10, TP11, TP12, TP13, TP14, TP15, TP16, TP17, TP18, TP19, TP3, TP4, TP5, TP6, TP7, TP8, TP9: TP0.4MM, particle SZ:TP0.4MM
- C12: device particle SZ:RESR0603A -> particle SZ:CAPC0805
- C13: device particle SZ:CAPC0201-N -> Particle:CAP_1; ITEM_NAME CAP CER 10uF 6.3V X5R 0603 10% Low ESR<70mohms -> CAP CER 0.1UF 16V X7R 0402 10%; ITEM_NUMBER PT-200209 -> PT-200649
- C14, C25, C28, C36, C47: device particle SZ:CAPC0201-N -> Particle:CAP_1; ITEM_NAME CAP CER 10uF 6.3V X5R 0603 10% Low ESR<70mohms -> (none); ITEM_NUMBER PT-200209 -> (none)
- C20: device particle SZ:CAPC0201-N -> Particle:CAP_1; ITEM_NAME CAP CER 10uF 6.3V X5R 0603 10% Low ESR<70mohms -> CAP CER 1000PF 50V X7R 0402 10%; ITEM_NUMBER PT-200209 -> (none)
- C22: device particle SZ:CAPC0201-N -> Particle:CAP_1; ITEM_NAME CAP CER 10uF 6.3V X5R 0603 10% Low ESR<70mohms -> CAP CER 10PF 5% 50V C0G/NP0 0402; ITEM_NUMBER PT-200209 -> 120-00038
- C26: device particle SZ:CAPC0603 -> particle SZ:CAPC0805
- L1, L3: device Particle:INDUCTOR-SPARKFUNINDUCTOR-2520 -> Particle:INDUCTOR-SPARKFUNVLS3012ET-4R7M
- R14, R23, R24, R28, R4, R5, R6: device particle SZ:RESR0201-N -> Spark:R-US_
- R16: value 100K -> 1M; device particle SZ:RESR0201-N -> Spark:R-US_
- R17: value 18K -> 24K; device particle SZ:RESR0201-N -> Spark:R-US_
- R34: value 49.9K -> 31.2K
- R35: value 27.4K -> 5.49K
- R8: value 510K -> 1M; device particle SZ:RESR0201-N -> Spark:R-US_
- R9: value 91K -> 180K; device particle SZ:RESR0201-N -> Spark:R-US_
- U1: value BQ24195 -> BQ24195L; device ELEKTRA-PMIC v0.3-35X22.86-0.8-0402:ELECTRON_BQ24298RTWR -> electron:BQ24298RTWR; ITEM_NAME (none) -> IC BATT CHG LI-ION 1CELL 24VQFN 2.5A CHG CURRENT; ITEM_NUMBER (none) -> 150-00013
- renumbered U2 to U$3, U3 to U6
Connections:
- removed net 3V3_AUX: C10.1, J2.2, R11.1, R12.1, U5.VOUT
- removed net EN_AUX: J2.7, R1.1, U5.ON
- removed net N$1: J2.3
- removed net N$10: J2.4
- removed net N$18: C7.1, U5.CT
- removed net N$20: R11.2, U5.QOD
- new net 5VDC: J2.3, J2.4
- net 3V3: now also C14.P$2, J2.2; no longer C14.1, U5.VIN
- net ENABLE: now also C25.P$2; no longer C25.1
- net GND: now also C13.P$1, C20.P$1, C22.P$1, C25.P$1, C36.P$1, C47.P$1, TP10.1, TP11.1, TP12.1, TP13.1, TP14.1, TP15.1, TP16.1, TP17.1, TP18.1, TP19.1, TP3.1, TP4.1, TP5.1, TP6.1, TP7.1, TP8.1, TP9.1; no longer C10.2, C13.2, C20.2, C22.2, C25.2, C36.2, C47.2, C7.2, R1.2, R12.2, R13.2, U$1.TP, U$2.TP, U$4.TP, U$5.TP, U5.GND
- net N$15: no longer R13.1
- net N$19: now also C36.P$2; no longer C36.1
- net N$21: now also C47.P$2; no longer C47.1
- net N$4: now also U1.!PG; no longer U1.D-
- net N$5: now also C14.P$1; no longer C14.2
- net N$6: now also C28.P$1; no longer C28.2
- net N$7: now also U1.PSEL; no longer U1.D+
- net REGN: now also J2.7; no longer J2.8
- net TS: now also U1.!QON, U1.TS; no longer U1.TS1, U1.TS2
- net VCC: now also C28.P$2; no longer C28.1
- net VSYS: now also C13.P$2, C20.P$2, C22.P$2; no longer C13.1, C20.1, C22.1
Other:
- note added: "Minimum Load is 200ma"
- note removed: "Reserve 5VDC interface"
- moved on the sheet: C101, C16, C18, C19, C23, C24, C27, C29, R16, R17, R24, R8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
