File: PM-BAT/v0.4/PM-BAT v0.4-35X22.86.brd (EAGLE design)
At the start: 35 x 22.9 mm, 87 parts, among them J1 M13PTH-CST-R, J2 M12PTH-CST-R, U1 BQ24195, U2 TPS63020, U3 TPS631011, U4 MAX1704X, U5 TPS22918

Commit message: update
change the name as PM-BAT
Parts:
- removed U4: MAX1704X, SparkFun-PowerIC:TDFN-8
- added U6: SPARKFUN-POWERIC_MAX1704X, ELEKTRA-PMIC v0.3-35X22.86-0.8-0402:SPARKFUN-POWERIC_TDFN-8
- moved R30 0.07 mm to (31.3, 10.1), turned to 180 degrees
Connections:
- net !FUEL-INT: now also U6.5; no longer U4.5
- net GND: now also U6.1, U6.4, U6.6, U6.EP; no longer U4.1, U4.4, U4.6, U4.EP
- net N$48: now also U6.3; no longer U4.3
- net N$49: now also U6.2; no longer U4.2
- net SCL: now also U6.7; no longer U4.7
- net SDA: now also U6.8; no longer U4.8
Routing:
- net SCL: track 31.3 -> 29.1 mm
- net GND: vias 153 -> 152
Other:
- board text added: "PM-BAT v0.4"
- board text removed: "ELEKTRA-PMIC v0.4"
