File: PM_DC/V0.3/PM_DC_v0.3.brd (EAGLE design)
At the start: 35 x 22.9 mm, 49 parts, among them J1 M13PTH-CST-R, J2 M12PTH-CST-R, U2 LMR14030, U3 MP1601GTF-Z, U5 TPS22918

Commit message: update
output gerber for MO DFM
Parts:
- C13: value nc -> 680pF
- R3: value 82K -> 76.8K
- R4: value 82K -> 100K
- R5: value 39.2K -> 44.2K
- R9: value 200K -> 0R
Routing:
- net GND: track 109.0 -> 123.1 mm
Other:
- board text added: "U2"
