File: PM-BAT/PM-BAT-V0.5-DXF for shielding case/PM-BAT v0.5-35X22.86-DXF.brd (EAGLE design)
At the start: 35 x 22.9 mm, 88 parts, among them J1 M13PTH-CST-R, J2 M12PTH-CST-R, U1 BQ24195, U2 TPS63020, U3 TPS631011, U5 TPS22918, U6 SPARKFUN-POWERIC_MAX1704X

Commit message: update
update  and output DXF for DFM
Routing:
- net GND: track 223.1 -> 18.2 mm, vias 171 -> 0
- net 3V3: track 96.6 -> 1.27 mm, vias 18 -> 0
- net VCC: track 60.7 -> 5.08 mm, vias 12 -> 0
- net VIN: track 54.3 -> 5.08 mm, vias 12 -> 0
- net VBAT: track 43.0 -> 3.81 mm, vias 21 -> 0
- net EN_AUX: track 28.5 -> 0.00 mm, vias 1 -> 0
- net SCL: track 29.1 -> 1.27 mm, vias 3 -> 0
- net REGN: track 27.4 -> 0.00 mm, vias 2 -> 0
- net SDA: track 25.6 -> 1.27 mm, vias 2 -> 0
- net !FUEL-INT: track 25.4 -> 1.27 mm, vias 2 -> 0
- net 3V3_AUX: track 23.5 -> 0.00 mm, vias 5 -> 0
- net PG: track 23.9 -> 1.27 mm, vias 1 -> 0
- net N$21: track 22.4 -> 0.00 mm, vias 2 -> 0
- net ENABLE: track 22.4 -> 1.27 mm, vias 3 -> 0
- net VSYS: track 18.9 -> 0.00 mm, vias 17 -> 0
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- removed copper zone on layer 1, net 3V3
- removed copper zone on layer 15, net 3V3
- removed copper zone on layer 16, net 3V3
- removed copper zone on layer 1, net 3V3_AUX
- removed copper zone on layer 15, net 3V3_AUX
- removed copper zone on layer 16, net 3V3_AUX
- removed copper zone on layer 1, net GND
- removed copper zone on layer 15, net GND
- removed copper zone on layer 16, net GND
- removed copper zone on layer 1, net N$11
- removed copper zone on layer 1, net N$12
- removed copper zone on layer 1, net N$16
- removed copper zone on layer 1, net N$17
- removed copper zone on layer 1, net N$3
- removed copper zone on layer 1, net SW1
- removed copper zone on layer 1, net VBAT
- removed copper zone on layer 15, net VBAT
- removed copper zone on layer 16, net VBAT
- removed copper zone on layer 1, net VCC
- removed copper zone on layer 15, net VCC
- removed copper zone on layer 16, net VCC
- removed copper zone on layer 1, net VIN
- removed copper zone on layer 15, net VIN
- removed copper zone on layer 16, net VIN
- removed copper zone on layer 1, net VSYS
- removed copper zone on layer 15, net VSYS
- removed copper zone on layer 16, net VSYS
Other:
- board text removed: "B4"
- board text removed: "P3"
- board text removed: "T1"
