File: PM-BAT/V0.5/PM-BAT v0.5-35X22.86.brd (EAGLE design)
At the start: 35 x 22.9 mm, 88 parts, among them J1 M13PTH-CST-R, J2 M12PTH-CST-R, U1 BQ24195, U2 TPS63020, U3 TPS631011, U5 TPS22918, U6 SPARKFUN-POWERIC_MAX1704X

Commit message: upload xydate and placement and update based test
Parts:
- C14, C28: value NC -> 47pF
- R13: value 100K/NC -> 100K
- R16: value 100K -> NC
- R17: value 18K -> 0R
- R18: value 10K -> NC
- R23: value 1M -> NC
- R24: value NC -> 1M
- R28: value 1M -> 100K
Other:
- board text added: "CON1"
- board text added: "CON2"
- board text added: "L1"
- board text added: "L3"
- board text added: "SHLD"
- board text removed: "NR3015T2R2M"
